Commit message: rearrangement of folders and deletion of unused files

File: ws/src/frida_description/urdf/urdf/FRIDA.urdf.xacro (robot description, xacro)
@@ -2,5 +2,5 @@
 <robot xmlns:xacro="http://www.ros.org/wiki/xacro" name="FRIDA">
 <!-- Properties -->
-<xacro:property name="mesh_path" value="package://frida_description/urdf/FRIDAurdf/meshes/" />
+<xacro:property name="mesh_path" value="package://frida_description/urdf/meshes/" />
 <xacro:property name="material_rgba" value="0.792 0.820 0.933 1" />
 <xacro:property name="lidar_rgba" value="0.102 0.102 0.102 1" />

Commit message: minor changes to urdf

File: ws/src/frida_description/urdf/urdf/FRIDA.urdf.xacro (robot description, xacro)
@@ -1,4 +1,4 @@
 <?xml version="1.0"?>
-<robot xmlns:xacro="http://www.ros.org/wiki/xacro" name="FRIDA">
+<robot name="FRIDA" xmlns:xacro="http://www.ros.org/wiki/xacro">
 <!-- Properties -->
 <xacro:property name="mesh_path" value="package://frida_description/urdf/meshes/" />
@@ -63,5 +63,5 @@
   <link name="left_wheel">
     <inertial>
-      <origin xyz="-0.1875 0.034916320504547 0.256" rpy="0 0 0" />
+      <origin xyz="-2.77555756156289E-17 0 -0.0389999999999999" rpy="0 0 0" />
       <mass value="0.528918539158378" />
       <inertia ixx="0.000631308353030454" ixy="-4.50512202234995E-20" ixz="-1.22382015150358E-21"
@@ -85,5 +85,5 @@
   </link>
   <joint name="leftwheel" type="continuous">
-    <origin xyz="0.11226 0.09 0.0025837" rpy="-1.5708 0 0" />
+    <origin xyz="-0.075244 0.205 0.0375" rpy="-1.5708 0 0" />
     <parent link="base_link" />
     <child link="left_wheel" />
@@ -93,7 +93,7 @@
   <link name="camera_link">
     <visual>
-      <origin xyz="0.0 0.0 0.5" rpy="0 0 0" />
+      <origin xyz="0 0 0" rpy="0 0 0" />
       <geometry>
-        <mesh filename="${mesh_path}camera.STL" />
+        <mesh filename="${mesh_path}intel_realsense.STL" />
       </geometry>
       <material name="">
@@ -103,5 +103,5 @@
   </link>
   <joint name="camera_joint" type="fixed">
-    <origin xyz="0.0 0.0 0.5" rpy="0 0 0" />
+    <origin xyz="0.06478 0 0.55626" rpy="0 0 0" />
     <parent link="base_link" />
     <child link="camera_link" />
@@ -109,8 +109,14 @@
   <!-- Lidar Sensor -->
   <link name="lidar_link">
+  <inertial>
+      <origin xyz="-1.38777878078145E-17 -3.38181918277552E-34 0.0125" rpy="0 0 0" />
+      <mass value="0.0962112750161874" />
+      <inertia ixx="3.44757068808005E-05" ixy="1.3254524700622E-52"  ixz="-6.00991536754997E-37"
+               iyy="3.44757068808005E-05" iyz="8.13422838622583E-38" izz="5.89294059474148E-05" />
+  </inertial>
     <visual>
-      <origin xyz="0.0 0.0 0.4" rpy="0 0 0" />
+      <origin xyz="0 0 0" rpy="0 0 0" />
       <geometry>
-        <mesh filename="${mesh_path}lidar.STL" />
+        <mesh filename="${mesh_path}LIDAR.STL" />
       </geometry>
       <material name="">
@@ -124,3 +130,23 @@
     <child link="lidar_link" />
   </joint>
+<!-- external Xarm6 attachment
+  <xacro:arg name="prefix" default="" />
+  <xacro:arg name="add_gripper" default="false" />
+  <xacro:arg name="add_vacuum_gripper" default="false" />
+  <xacro:arg name="robot_type" default="xarm" />
+  <xacro:arg name="model1300" default="false" />
+  <xacro:arg name="add_realsense_d435i" default="false" />
+  <xacro:arg name="add_d435i_links" default="false" />
+  <xacro:arg name="robot_sn" default="" />
+  <xacro:arg name="dof" default="6" />
+  <xacro:include filename="$(find xarm_description)/urdf/xarm_device_macro.xacro" />
+  <xacro:xarm_device prefix="$(arg prefix)" dof="$(arg dof)" attach_to="BaseBrazo" model1300="$(arg model1300)" add_gripper="$(arg add_gripper)" add_vacuum_gripper="$(arg add_vacuum_gripper)" add_realsense_d435i="$(arg add_realsense_d435i)" add_d435i_links="$(arg add_d435i_links)" robot_sn="$(arg robot_sn)" />
+  <xacro:include filename="$(find robot_description)/urdf/gripper/gripper.urdf.xacro" />
+  <xacro:include filename="$(find robot_description)/urdf/gripper/gripperP.urdf.xacro" />
+  <xacro:include filename="$(find robot_description)/urdf/gripper/gripperFakeSF.urdf.xacro" />
+  <xacro:include filename="$(find robot_description)/urdf/gripper/gripperSF.urdf.xacro" />
+  <xacro:load_gripperSF attach_to="$(arg prefix)link_eef" xyz="0 0 0.007" rpy="-1.57 0 2.3554" />
+  <xacro:include filename="$(find robot_description)/urdf/camera.urdf.xacro" />
+  <xacro:load_camera name="Cam1" attach_to="Base_Gripper" x="0.068098" y="-0.035446" z="0.0" r_p="-0.785398" r_r="1.5707" r_y="0.0" />
+-->
 </robot>
